File: RPi_CM4_Breakout.kicad_pcb (KiCad board)
At the start: 2 copper layers, 48 x 72 mm, 23 parts, among them J1 RPi_pin, J2 UJC-HP-3-SMT-TR, J3 Conn_01x04_Female, J4 Conn_01x04_Female, J5 Conn_01x04_Female, J6 Conn_01x04_Female, U1 74LVC1G07

Commit message: fix: 調整
Parts:
- moved R4 1.75 mm to (195.6, 53.3)
Routing:
- net Net-(J2-PadB5): track 6.92 -> 7.86 mm
- net +3V3: track 195.7 -> 196.3 mm
- net GND: vias 61 -> 78
Other:
- board text added: "J7"
- board text added: "J8"
- board text added: "ver 0.2 (2021.08.27)"
- board text removed: "ver 0.1 (2021.08.16)"

Commit message: fix: LED ドライバのパッケージを SOT753 に変更
Parts:
- U1: footprint Package_TO_SOT_SMD:SOT-353_SC-70-5_Handsoldering -> CMIO:SOT-753
- moved U1 0.37 mm to (214.1, 52.1), turned to -90 degrees
