File: RPi_CM4_Breakout.kicad_sch (KiCad schematic)
At the start: 23 parts, among them J1 RPi_pin, J2 UJC-HP-3-SMT-TR, J3 Conn_01x04_Female, J4 Conn_01x04_Female, J5 Conn_01x04_Female, J6 Conn_01x04_Female, U1 74LVC1G07

Commit message: fix: LED ドライバのパッケージを SOT753 に変更
Parts:
- U1: footprint Package_TO_SOT_SMD:SOT-353_SC-70-5_Handsoldering -> CMIO:SOT-753
Changed lines of the file:
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@@
     (property "Reference" "U1" (id 0) (at 155.575 37.6894 0))
     (property "Value" "74LVC1G07" (id 1) (at 155.575 40.4645 0))
-    (property "Footprint" "Package_TO_SOT_SMD:SOT-353_SC-70-5_Handsoldering" (id 2) (at 156.21 44.45 0)
+    (property "Footprint" "CMIO:SOT-753" (id 2) (at 156.21 44.45 0)
       (effects (font (size 1.27 1.27)) hide)
     )
@@
     )
     (path "/e39ff249-1fd2-40b0-a7fa-944d830b3327"
-      (reference "U1") (unit 1) (value "74LVC1G07") (footprint "Package_TO_SOT_SMD:SOT-353_SC-70-5_Handsoldering")
-    )
-  )
+      (reference "U1") (unit 1) (value "74LVC1G07") (footprint "CMIO:SOT-753")
+    )
+  )
